Commit message: Keep simulator setup aligned for graph SLAM
The local simulator tweaks need to sit on top of the graph_slam package that landed on origin/main, so this preserves the RViz, sensor pose, and track generator fixes while making the branch pushable again.

Constraint: origin/main already contains the graph_slam package commit

Rejected: Add a merge commit | the local and remote changes are disjoint, so rebasing keeps history simpler

Confidence: high

Scope-risk: moderate

Reversibility: clean

Tested: git rebase origin/main

Not-tested: ROS build or runtime simulation

File: eufs_sim/eufs_racecar/robots/eufs/robot.urdf.xacro (robot description, xacro)
@@ -47,6 +47,7 @@
     </xacro:sensor_gps>
     <xacro:VLP-16R parent="chassis" name="velodyne" topic="/velodyne_points" hz="10" active="$(arg simulate_perception)">
-        <origin xyz="1.6 0.0 0.25" rpy="0 ${1*M_PI/180.0} 0"/>
+        <origin xyz="-0.15 0.0 0.79" rpy="0 ${1*M_PI/180.0} 0"/>
         <!--<origin xyz="-0.15 0.0 0.79" rpy="0 ${1*M_PI/180.0} 0"/>-->
+        <!--<origin xyz="1.6 0.0 0.25" rpy="0 ${1*M_PI/180.0} 0"/>-->
     </xacro:VLP-16R>
     <xacro:zed_camera parent="chassis" prefix="zed" active="$(arg simulate_perception)">

File: eufs_sim/eufs_sensors/urdf/VLP-16R.urdf.xacro (robot description, xacro)
@@ -2,5 +2,17 @@
 <robot xmlns:xacro="http://www.ros.org/wiki/xacro" name="VLP-16">
   <xacro:property name="M_PI" value="3.1415926535897931" />
-  <xacro:macro name="VLP-16R" params="*origin parent:=base_footprint name:=velodyne active topic:=/velodyne_points hz:=10 lasers:=40 samples:=350 min_range:=0.2 max_range:=100.0 noise:=0.008 min_angle:=-2 max_angle:=2">
+  <xacro:macro
+    name="VLP-16R"
+    params="*origin parent:=base_footprint
+            name:=velodyne active
+            topic:=/velodyne_points
+            hz:=10
+            lasers:=40
+            samples:=350
+            min_range:=0.2
+            max_range:=100.0
+            noise:=0.008
+            min_angle:=-2
+            max_angle:=2">
     <joint name="${name}_base_mount_joint" type="fixed">
       <xacro:insert_block name="origin" />
