Commit message: Wire perception into sim launch, fix pipeline traps found in e2e verification
- simulation.launch.py: include eufs_perception_baseline behind perception:=true
  (venv/conda python auto-detect); fail fast on perception:=true +
  launch_group:=no_perception (duplicate /cones publishers + starved fusion);
  warn when defaults leave /cones with no publisher at all.
- robot.urdf.xacro: VLP-16 lasers=16 (macro default was 40) and move the lidar
  to the real car's nose-cone mount (1.6, 0, 0.25).
- sim_ellipse_d: ekf_rate default 25 -> 200 Hz to match the real Ellipse-D
  output; expose ekf_rate as an ins_pipeline launch argument.
- perception_baseline: model_path -> in-repo models/fsoco_yolov8n/weights
  (weights gitignored), device cuda:0.

Verified end-to-end on small_track: camera 15.8Hz -> YOLO 15.8Hz -> fusion
/cones 13.8Hz -> graph SLAM landmarks 6->20 while driving.

Co-Authored-By: Claude Fable 5 (1M context) <noreply@anthropic.com>

File: eufs_sim/eufs_racecar/robots/eufs/robot.urdf.xacro (robot description, xacro)
@@ -46,8 +46,9 @@
         <origin xyz="0.0 0.0 0.4" rpy="0 0 0"/>
     </xacro:sensor_gps>
-    <xacro:VLP-16R parent="chassis" name="velodyne" topic="/velodyne_points" hz="10" active="$(arg simulate_perception)">
-        <origin xyz="-0.15 0.0 0.79" rpy="0 ${1*M_PI/180.0} 0"/>
-        <!--<origin xyz="-0.15 0.0 0.79" rpy="0 ${1*M_PI/180.0} 0"/>-->
-        <!--<origin xyz="1.6 0.0 0.25" rpy="0 ${1*M_PI/180.0} 0"/>-->
+    <!-- Real car: VLP-16 (16 channels) mounted on the nose cone.
+         lasers must be passed explicitly — the VLP-16R macro default is 40. -->
+    <xacro:VLP-16R parent="chassis" name="velodyne" topic="/velodyne_points" hz="10" lasers="16" active="$(arg simulate_perception)">
+        <origin xyz="1.6 0.0 0.25" rpy="0 ${1*M_PI/180.0} 0"/>
+        <!-- main-hoop mount (previous): <origin xyz="-0.15 0.0 0.79" rpy="0 ${1*M_PI/180.0} 0"/> -->
     </xacro:VLP-16R>
     <xacro:zed_camera parent="chassis" prefix="zed" active="$(arg simulate_perception)">
