Commit message: feat: Updated Perception Pipeline wrt IIT Bombay paper

File: eufs_sim/eufs_racecar/robots/eufs/robot.urdf.xacro (robot description, xacro)
@@ -47,5 +47,5 @@
     </xacro:sensor_gps>
     <xacro:VLP-16R parent="chassis" name="velodyne" topic="/velodyne_points" hz="10" lasers="16" active="$(arg simulate_perception)">
-        <origin xyz="1.4 0.0 0.38" rpy="0 ${8*M_PI/180.0} 0"/>
+        <origin xyz="1.8 0.0 0.2" rpy="0 0 0"/>
     </xacro:VLP-16R>
     <!-- <xacro:VLP-16R parent="chassis" name="velodyne" topic="/velodyne_points" hz="10" lasers="16" active="$(arg simulate_perception)"> -->
