Commit message: Add YOLO perception fusion pipeline

File: eufs_sim/eufs_plugins/urdf/eufs_plugins.gazebo.xacro (robot description, xacro)
@@ -53,7 +53,10 @@
       <recolor_config>$(arg recolor_config)</recolor_config>
       <groundTruthConesTopicName>/ground_truth/cones</groundTruthConesTopicName>
+      <groundTruthConeMarkersTopicName>/ground_truth/cones/viz</groundTruthConeMarkersTopicName>
       <groundTruthTrackTopicName>/ground_truth/track</groundTruthTrackTopicName>
+      <groundTruthTrackMarkersTopicName>/ground_truth/track/viz</groundTruthTrackMarkersTopicName>
       <simulatePerception>$(arg simulate_perception)</simulatePerception>
       <perceptionConesTopicName>/cones</perceptionConesTopicName>
+      <perceptionConeMarkersTopicName>/cones/viz</perceptionConeMarkersTopicName>
       <perceptionCameraDepthNoiseParameterA>0.01</perceptionCameraDepthNoiseParameterA>
       <perceptionCameraDepthNoiseParameterB>0.5</perceptionCameraDepthNoiseParameterB>
@@ -72,4 +75,5 @@
       <recolorConfig>cone_recolor.yaml</recolorConfig>
       <cameraConesTopicName>/camera_0/cones</cameraConesTopicName>
+      <cameraConeMarkersTopicName>/camera_0/cones/viz</cameraConeMarkersTopicName>
       <perceptionCameraDepthNoiseParameterA>0.01</perceptionCameraDepthNoiseParameterA>
       <perceptionCameraDepthNoiseParameterB>0.5</perceptionCameraDepthNoiseParameterB>
@@ -86,4 +90,5 @@
       <recolorConfig>cone_recolor.yaml</recolorConfig>
       <cameraConesTopicName>/camera_1/cones</cameraConesTopicName>
+      <cameraConeMarkersTopicName>/camera_1/cones/viz</cameraConeMarkersTopicName>
       <perceptionCameraDepthNoiseParameterA>0.01</perceptionCameraDepthNoiseParameterA>
       <perceptionCameraDepthNoiseParameterB>0.5</perceptionCameraDepthNoiseParameterB>

File: eufs_sim/eufs_racecar/robots/eufs/robot.urdf.xacro (robot description, xacro)
@@ -46,9 +46,16 @@
         <origin xyz="0.0 0.0 0.4" rpy="0 0 0"/>
     </xacro:sensor_gps>
-    <xacro:VLP-16R parent="chassis" name="velodyne" topic="/velodyne_points" hz="10" active="$(arg simulate_perception)">
-        <origin xyz="-0.15 0.0 0.79" rpy="0 ${1*M_PI/180.0} 0"/>
-        <!--<origin xyz="-0.15 0.0 0.79" rpy="0 ${1*M_PI/180.0} 0"/>-->
-        <!--<origin xyz="1.6 0.0 0.25" rpy="0 ${1*M_PI/180.0} 0"/>-->
+    <xacro:VLP-16R parent="chassis" name="velodyne" topic="/velodyne_points" hz="10" lasers="16" active="$(arg simulate_perception)">
+        <origin xyz="1.4 0.0 0.38" rpy="0 ${8*M_PI/180.0} 0"/>
     </xacro:VLP-16R>
+    <!-- <xacro:VLP-16R parent="chassis" name="velodyne" topic="/velodyne_points" hz="10" lasers="16" active="$(arg simulate_perception)"> -->
+        <!-- <origin xyz="1.1 0.0 0.38" rpy="0 ${8*M_PI/180.0} 0"/> -->
+    <!-- </xacro:VLP-16R> -->
+    <!-- <xacro:VLP-16R parent="chassis" name="velodyne_compare" topic="/velodyne_compare_points" hz="10" lasers="16" active="$(arg simulate_perception)">
+        <origin xyz="1.35 0.0 -0.14" rpy="0 ${1*M_PI/180.0} 0"/>
+    </xacro:VLP-16R> -->
+    <!-- <xacro:VLP-16R parent="chassis" name="velodyne" topic="/velodyne_points" hz="10" lasers="16" active="$(arg simulate_perception)">
+        <origin xyz="0 0.0 0" rpy="0 ${1*M_PI/180.0} 0"/>
+    </xacro:VLP-16R> -->
     <xacro:zed_camera parent="chassis" prefix="zed" active="$(arg simulate_perception)">
         <origin xyz="-0.08 0.0 0.76" rpy="0 0 0"/>

File: eufs_sim/eufs_sensors/urdf/zed.urdf.xacro (robot description, xacro)
@@ -90,4 +90,16 @@
               <remapping>/${prefix}_left/image_raw:=/${prefix}/left/image_rect_color</remapping>
               <remapping>/${prefix}_left/camera_info:=/${prefix}/left/camera_info</remapping>
+              <qos>
+                <topic name="/${prefix}/left/image_rect_color">
+                  <publisher>
+                    <reliability>reliable</reliability>
+                  </publisher>
+                </topic>
+                <topic name="/${prefix}/left/camera_info">
+                  <publisher>
+                    <reliability>reliable</reliability>
+                  </publisher>
+                </topic>
+              </qos>
             </ros>
             <camera_name>${prefix}_left</camera_name>
@@ -125,4 +137,16 @@
               <remapping>/${prefix}_right/image_raw:=/${prefix}/right/image_rect_color</remapping>
               <remapping>/${prefix}_right/camera_info:=/${prefix}/right/camera_info</remapping>
+              <qos>
+                <topic name="/${prefix}/right/image_rect_color">
+                  <publisher>
+                    <reliability>reliable</reliability>
+                  </publisher>
+                </topic>
+                <topic name="/${prefix}/right/camera_info">
+                  <publisher>
+                    <reliability>reliable</reliability>
+                  </publisher>
+                </topic>
+              </qos>
             </ros>
             <camera_name>${prefix}_right</camera_name>
