Commit message: .

File: eufs_sim/eufs_plugins/urdf/eufs_plugins.gazebo.xacro (robot description, xacro)
@@ -26,4 +26,12 @@
       <groundTruthCarStateTopic>/ground_truth/state</groundTruthCarStateTopic>
       <localisationCarStateTopic>/odometry_integration/car_state</localisationCarStateTopic>
+      <!-- Drifting odometry for the localisation car state (GT stays on
+           groundTruthCarStateTopic). Set driftOdometry to false to restore the
+           noise-model behaviour. -->
+      <driftOdometry>true</driftOdometry>
+      <driftVelocityBias>0.02</driftVelocityBias>
+      <driftYawRateBias>0.01</driftYawRateBias>
+      <driftVelocityNoise>0.05</driftVelocityNoise>
+      <driftYawRateNoise>0.01</driftYawRateNoise>
       <wheelSpeedsTopicName>/ros_can/wheel_speeds</wheelSpeedsTopicName>
       <groundTruthWheelSpeedsTopicName>/ground_truth/wheel_speeds</groundTruthWheelSpeedsTopicName>

File: eufs_sim/eufs_racecar/robots/ads-dv/robot.urdf.xacro (robot description, xacro)
@@ -5,5 +5,5 @@
     <!-- ***************** -->
     <!--  Load the config file  -->
-    <xacro:property name="config" value="${load_yaml('$(arg config_file)')}"/>
+    <xacro:property name="config" value="${xacro.load_yaml('$(arg config_file)')}"/>
     <!-- ***************** -->
     <!-- Global parameters -->

File: eufs_sim/eufs_racecar/robots/eufs/robot.urdf.xacro (robot description, xacro)
@@ -5,5 +5,5 @@
     <!-- ***************** -->
     <!--  Load the config file  -->
-    <xacro:property name="config" value="${load_yaml('$(arg config_file)')}"/>
+    <xacro:property name="config" value="${xacro.load_yaml('$(arg config_file)')}"/>
     <!-- ***************** -->
     <!-- Global parameters -->

File: eufs_sim/eufs_racecar/urdf/wheels.urdf.xacro (robot description, xacro)
@@ -6,4 +6,7 @@
     <!-- Parameters -->
     <!-- ********** -->
+    <material name="tire_mat">
+      <color rgba="0.12 0.12 0.12 1.0"/>
+    </material>
     <xacro:property name="degrees_90" value="1.5708"/>
     <xacro:property name="wheel_mass" value="10.0"/>

Commit message: Import the full Formula Student planning pipeline

File: eufs_sim/eufs_plugins/urdf/eufs_plugins.gazebo.xacro (robot description, xacro)
@@ -5,4 +5,18 @@
   <xacro:arg name="command_mode" default="acceleration"/>
   <xacro:arg name="pub_ground_truth" default="true"/>
+  <xacro:arg name="perception_camera_view_distance" default="15"/>
+  <xacro:arg name="perception_lidar_view_distance" default="100"/>
+  <xacro:arg name="perception_lidar_x_view_distance" default="20"/>
+  <xacro:arg name="perception_lidar_y_view_distance" default="20"/>
+  <xacro:arg name="perception_lidar_min_view_distance" default="1"/>
+  <xacro:arg name="perception_camera_min_view_distance" default="0.5"/>
+  <xacro:arg name="perception_camera_fov" default="2.09"/>
+  <xacro:arg name="perception_lidar_fov" default="3.141593"/>
+  <xacro:arg name="perception_lidar_on" default="true"/>
+  <xacro:arg name="perception_detection_probability" default="1.0"/>
+  <xacro:arg name="camera_cones_view_distance" default="13"/>
+  <xacro:arg name="camera_cones_min_view_distance" default="0.5"/>
+  <xacro:arg name="camera_cones_fov" default="2.09"/>
+  <xacro:arg name="camera_cones_detection_probability" default="1.0"/>
   <!-- Custom plugin which controls the car using a given vehicle model.
    It controls the car by setting its velocity and position
@@ -26,4 +40,12 @@
       <groundTruthCarStateTopic>/ground_truth/state</groundTruthCarStateTopic>
       <localisationCarStateTopic>/odometry_integration/car_state</localisationCarStateTopic>
+      <!-- Drifting odometry for the localisation car state (GT stays on
+           groundTruthCarStateTopic). Set driftOdometry to false to restore the
+           noise-model behaviour. -->
+      <driftOdometry>true</driftOdometry>
+      <driftVelocityBias>0.02</driftVelocityBias>
+      <driftYawRateBias>0.01</driftYawRateBias>
+      <driftVelocityNoise>0.05</driftVelocityNoise>
+      <driftYawRateNoise>0.01</driftYawRateNoise>
       <wheelSpeedsTopicName>/ros_can/wheel_speeds</wheelSpeedsTopicName>
       <groundTruthWheelSpeedsTopicName>/ground_truth/wheel_speeds</groundTruthWheelSpeedsTopicName>
@@ -40,23 +62,21 @@
     <plugin name="gz_ground_truth_cones" filename="libgazebo_ground_truth_cones.so">
       <alwaysOn>true</alwaysOn>
-      <updateRate>100.0</updateRate>
-      <cameraViewDistance>15</cameraViewDistance>
-      <lidarViewDistance>100</lidarViewDistance>
-      <lidarXViewDistance>20</lidarXViewDistance>
-      <lidarYViewDistance>20</lidarYViewDistance>
-      <lidarMinViewDistance>1</lidarMinViewDistance>
-      <cameraFOV>2.09</cameraFOV><!--120 degrees-->
-      <cameraMinViewDistance>0.5</cameraMinViewDistance>
-      <lidarFOV>3.141593</lidarFOV><!-- 180 degrees-->
-      <lidarOn>true</lidarOn><!--If false, we only simulate camera measurements-->
+      <updateRate>20.0</updateRate>
+      <cameraViewDistance>$(arg perception_camera_view_distance)</cameraViewDistance>
+      <lidarViewDistance>$(arg perception_lidar_view_distance)</lidarViewDistance>
+      <lidarXViewDistance>$(arg perception_lidar_x_view_distance)</lidarXViewDistance>
+      <lidarYViewDistance>$(arg perception_lidar_y_view_distance)</lidarYViewDistance>
+      <lidarMinViewDistance>$(arg perception_lidar_min_view_distance)</lidarMinViewDistance>
+      <cameraFOV>$(arg perception_camera_fov)</cameraFOV><!-- radians -->
+      <cameraMinViewDistance>$(arg perception_camera_min_view_distance)</cameraMinViewDistance>
+      <lidarFOV>$(arg perception_lidar_fov)</lidarFOV><!-- radians -->
+      <lidarOn>$(arg perception_lidar_on)</lidarOn><!--If false, we only simulate camera measurements-->
       <trackFrame>map</trackFrame>
       <recolor_config>$(arg recolor_config)</recolor_config>
       <groundTruthConesTopicName>/ground_truth/cones</groundTruthConesTopicName>
-      <groundTruthConeMarkersTopicName>/ground_truth/cones/viz</groundTruthConeMarkersTopicName>
       <groundTruthTrackTopicName>/ground_truth/track</groundTruthTrackTopicName>
-      <groundTruthTrackMarkersTopicName>/ground_truth/track/viz</groundTruthTrackMarkersTopicName>
       <simulatePerception>$(arg simulate_perception)</simulatePerception>
       <perceptionConesTopicName>/cones</perceptionConesTopicName>
-      <perceptionConeMarkersTopicName>/cones/viz</perceptionConeMarkersTopicName>
+      <detectionProbability>$(arg perception_detection_probability)</detectionProbability>
       <perceptionCameraDepthNoiseParameterA>0.01</perceptionCameraDepthNoiseParameterA>
       <perceptionCameraDepthNoiseParameterB>0.5</perceptionCameraDepthNoiseParameterB>
@@ -69,11 +89,11 @@
       <alwaysOn>true</alwaysOn>
       <updateRate>15.0</updateRate>
-      <cameraViewDistance>13</cameraViewDistance>
-      <cameraFOV>2.09</cameraFOV><!--120 degrees-->
-      <cameraMinViewDistance>0.5</cameraMinViewDistance>
+      <cameraViewDistance>$(arg camera_cones_view_distance)</cameraViewDistance>
+      <cameraFOV>$(arg camera_cones_fov)</cameraFOV><!-- radians -->
+      <cameraMinViewDistance>$(arg camera_cones_min_view_distance)</cameraMinViewDistance>
       <cameraTF>0.204 0.074 0.706 0 0 0.79</cameraTF>
       <recolorConfig>cone_recolor.yaml</recolorConfig>
       <cameraConesTopicName>/camera_0/cones</cameraConesTopicName>
-      <cameraConeMarkersTopicName>/camera_0/cones/viz</cameraConeMarkersTopicName>
+      <detectionProbability>$(arg camera_cones_detection_probability)</detectionProbability>
       <perceptionCameraDepthNoiseParameterA>0.01</perceptionCameraDepthNoiseParameterA>
       <perceptionCameraDepthNoiseParameterB>0.5</perceptionCameraDepthNoiseParameterB>
@@ -84,11 +104,11 @@
       <alwaysOn>true</alwaysOn>
       <updateRate>15.0</updateRate>
-      <cameraViewDistance>13</cameraViewDistance>
-      <cameraFOV>2.09</cameraFOV><!--120 degrees-->
-      <cameraMinViewDistance>0.5</cameraMinViewDistance>
+      <cameraViewDistance>$(arg camera_cones_view_distance)</cameraViewDistance>
+      <cameraFOV>$(arg camera_cones_fov)</cameraFOV><!-- radians -->
+      <cameraMinViewDistance>$(arg camera_cones_min_view_distance)</cameraMinViewDistance>
       <cameraTF>0.204 -0.074 0.706 0.0 0.0 -0.79</cameraTF>
       <recolorConfig>cone_recolor.yaml</recolorConfig>
       <cameraConesTopicName>/camera_1/cones</cameraConesTopicName>
-      <cameraConeMarkersTopicName>/camera_1/cones/viz</cameraConeMarkersTopicName>
+      <detectionProbability>$(arg camera_cones_detection_probability)</detectionProbability>
       <perceptionCameraDepthNoiseParameterA>0.01</perceptionCameraDepthNoiseParameterA>
       <perceptionCameraDepthNoiseParameterB>0.5</perceptionCameraDepthNoiseParameterB>

File: eufs_sim/eufs_racecar/robots/eufs/robot.urdf.xacro (robot description, xacro)
@@ -5,5 +5,5 @@
     <!-- ***************** -->
     <!--  Load the config file  -->
-    <xacro:property name="config" value="${load_yaml('$(arg config_file)')}"/>
+    <xacro:property name="config" value="${xacro.load_yaml('$(arg config_file)')}"/>
     <!-- ***************** -->
     <!-- Global parameters -->
@@ -46,16 +46,10 @@
         <origin xyz="0.0 0.0 0.4" rpy="0 0 0"/>
     </xacro:sensor_gps>
+    <!-- Real car: VLP-16 (16 channels) mounted on the nose cone.
+         lasers must be passed explicitly — the VLP-16R macro default is 40. -->
     <xacro:VLP-16R parent="chassis" name="velodyne" topic="/velodyne_points" hz="10" lasers="16" active="$(arg simulate_perception)">
-        <origin xyz="1.8 0.0 0.2" rpy="0 0 0"/>
+        <origin xyz="1.6 0.0 0.25" rpy="0 ${1*M_PI/180.0} 0"/>
+        <!-- main-hoop mount (previous): <origin xyz="-0.15 0.0 0.79" rpy="0 ${1*M_PI/180.0} 0"/> -->
     </xacro:VLP-16R>
-    <!-- <xacro:VLP-16R parent="chassis" name="velodyne" topic="/velodyne_points" hz="10" lasers="16" active="$(arg simulate_perception)"> -->
-        <!-- <origin xyz="1.1 0.0 0.38" rpy="0 ${8*M_PI/180.0} 0"/> -->
-    <!-- </xacro:VLP-16R> -->
-    <!-- <xacro:VLP-16R parent="chassis" name="velodyne_compare" topic="/velodyne_compare_points" hz="10" lasers="16" active="$(arg simulate_perception)">
-        <origin xyz="1.35 0.0 -0.14" rpy="0 ${1*M_PI/180.0} 0"/>
-    </xacro:VLP-16R> -->
-    <!-- <xacro:VLP-16R parent="chassis" name="velodyne" topic="/velodyne_points" hz="10" lasers="16" active="$(arg simulate_perception)">
-        <origin xyz="0 0.0 0" rpy="0 ${1*M_PI/180.0} 0"/>
-    </xacro:VLP-16R> -->
     <xacro:zed_camera parent="chassis" prefix="zed" active="$(arg simulate_perception)">
         <origin xyz="-0.08 0.0 0.76" rpy="0 0 0"/>
