Commit message: perception: pace /cones off the LiDAR; make the Puck's resolution follow its rate
Three things, one theme: a number that looked independent was not.

/cones ran off the camera at 30 Hz. The LiDAR is the backbone -- it is what
measures where a cone is -- so the camera pace republished the same clusters two
extra times per cloud, each dressed in a fresh stamp, inviting a consumer to read
three independent measurements where there was one. Inverting it was nearly free,
because Scene already separated the two things that want different instants:
positions come from the cloud's own stamp and so need no compensation at all,
while pixels must line up with an image up to one bbox period old, so the
projection, and only the projection, time-travels back to the image stamp.
Skipping that would mis-associate real cones at range: 33 ms at 6.5 m/s is
0.21 m, about 20 px at 15 m against a cone roughly 30 px wide. Vision-only cones
are carried the other way, so the single header stamp is true for every cone in
the array rather than just for the clusters. Measured: /cones 10.00 Hz at 1.3 ms
jitter, locked to velodyne's 10.00, latency p90 ~83 ms.

VLP-16 horizontal resolution is forced by the rotation rate: the laser fires on a
fixed interval, so spinning faster spreads the same firings over more degrees.
The datasheet's 0.1/0.2/0.4 deg at 5/10/20 Hz falls out of that, and the tell is
that points/second is 288k at all three rates, matching the ~300k on the spec
sheet. The macro now takes hz alone and derives samples = 18000/hz. Carrying both
let them disagree, which is how ads-dv ended up asking for 0.45 deg at 10 Hz, a
sensor that does not exist, while silently taking the macro's 40-laser default
against the real 16. Verified: 5/10/20 Hz expand to exactly 0.1/0.2/0.4 deg.

The stereo pair now renders at one instant (multicamera), but that fix was aimed
at a bug that was not there. Every "right camera at half rate" reading this
session came from probes subscribing to both 2.7 MB streams from one Python
process, which cannot deserialise 2x30 Hz of them; the right callback starves and
reads ~15 Hz. Measured one topic per process, both cameras are at 29.41 Hz and
always were. A MultiThreadedExecutor does not help -- it is the GIL, not
scheduling. The multicamera sensor stays because stamp-identical-by-construction
is the right structure, but the comment crediting it with fixing a split is
retracted, along with the ray-count claim in VLP-16R.urdf.xacro.

That consumer limit is real for the perception node too, so stereo halves are now
paired by exact stamp instead of latest-wins. Under latest-wins the node would
hold a left and right up to 33 ms apart and hand them to ZNCC, which cannot tell
ego motion from depth: 0.21 m of the car's own travel reported as a confident
cone range. Measured: zncc 195/195 and 223/223 confirmed, 0 skew rejections.

Also: simulation.launch.py could not start perception at all. It still included
perception_baseline.launch.py by its pre-rebuild name and still forwarded
bbox_source, monocular_fallback_enabled and other tier-era arguments the new
interface does not declare, which fails the whole launch. Tests now cover both
halves of that contract, and the `--`-in-an-XML-comment trap that has broken this
build six times is a build-time test rather than my discipline.

Co-Authored-By: Claude Opus 4.8 (1M context) <noreply@anthropic.com>

File: eufs_sim/eufs_plugins/urdf/eufs_plugins.gazebo.xacro (robot description, xacro)
@@ -23,4 +23,13 @@
   <xacro:arg name="camera_cones_fov" default="2.09"/>
   <xacro:arg name="camera_cones_detection_probability" default="1.0"/>
+  <!-- Road-roughness vibration. On by default (unchanged behaviour), but it is
+       the loudest thing on the body attitude at speed, so turn it off to observe
+       the car's own physics. -->
+  <xacro:arg name="road_noise" default="true"/>
+  <!-- Procedural bump field; off by default so existing runs are unchanged. -->
+  <xacro:arg name="terrain" default="false"/>
+  <xacro:arg name="terrain_seed" default="7"/>
+  <xacro:arg name="terrain_density" default="0.02"/>
+  <xacro:arg name="terrain_height_mean" default="0.020"/>
   <!-- Custom plugin which controls the car using a given vehicle model.
    It controls the car by setting its velocity and position
@@ -56,5 +65,5 @@
            so the rigidly-attached IMU/camera/LiDAR feel it too. Set roadNoise
            to false to keep the car perfectly flat. -->
-      <roadNoise>true</roadNoise>
+      <roadNoise>$(arg road_noise)</roadNoise>
       <roadNoiseZ>0.010</roadNoiseZ><!-- vertical bounce stddev [m] at v_ref -->
       <roadNoiseRoll>0.006</roadNoiseRoll><!-- roll stddev [rad] at v_ref -->
@@ -65,12 +74,37 @@
       <!-- Acceleration load transfer: longitudinal accel pitches the body
            (accel = nose up, braking = dive), lateral accel rolls it outward in
-           a corner. Gains are rad per m/s^2 (~0.006 -> ~3.4 deg at 1 g). Raise
-           for a more dramatic lean; set loadTransfer false to disable. -->
+           a corner. How far it leans and how it gets there are properties of the
+           car, so they live in its vehicle config (the `suspension:` block in
+           robots/[car]/config*.yaml) alongside its mass and tyres, including
+           `load_transfer_to_tires`, which couples the transfer into tyre grip.
+           Only the safety clamps are here. -->
       <loadTransfer>true</loadTransfer>
-      <loadTransferRollGain>0.010</loadTransferRollGain><!-- roll per lateral accel [rad/(m/s^2)] -->
-      <loadTransferPitchGain>0.010</loadTransferPitchGain><!-- pitch per long. accel [rad/(m/s^2)] -->
-      <loadTransferTau>0.15</loadTransferTau><!-- suspension response time [s] -->
       <loadTransferMaxRoll>0.12</loadTransferMaxRoll><!-- clamp [rad] (~6.9 deg) -->
       <loadTransferMaxPitch>0.12</loadTransferMaxPitch><!-- clamp [rad] -->
+      <!-- Procedural bump field. Unlike roadNoise above, these are real geometry
+           inserted into the world: the LiDAR ray-traces them and the cameras see
+           them, and the car's z/roll/pitch come from the terrain height under
+           each wheel, so the bump in the point cloud is the bump the car climbs.
+           Bumps are a function of position, so the same seed is the same track
+           every run and driving a line twice hits the same bumps twice.
+           Defaults are gentle asphalt undulation (~2 cm). Raise terrainHeightMean
+           to stress ground-plane RANSAC and the INS; set terrain false for the
+           perfectly flat floor. -->
+      <terrain>$(arg terrain)</terrain>
+      <terrainSeed>$(arg terrain_seed)</terrainSeed>
+      <terrainDensity>$(arg terrain_density)</terrainDensity><!-- bumps per m^2 -->
+      <terrainHeightMean>$(arg terrain_height_mean)</terrainHeightMean><!-- peak height [m] -->
+      <terrainHeightSigma>0.010</terrainHeightSigma><!-- height stddev [m] -->
+      <terrainHeightMin>0.004</terrainHeightMin><!-- floor on the height draw [m] -->
+      <terrainRadiusMin>0.25</terrainRadiusMin><!-- footprint radius [m] -->
+      <terrainRadiusMax>0.60</terrainRadiusMax>
+      <!-- Bumps are grown within this distance of a track cone: the car only
+           drives between the cones, so that is the only ground a bump can
+           matter on, and covering the rest costs thousands of them for nothing. -->
+      <terrainTrackMargin>3.5</terrainTrackMargin><!-- [m] from any cone -->
+      <terrainMaxBumps>600</terrainMaxBumps><!-- refuse to build a world that kills gzserver -->
+      <!-- Fallback area, used only if the world has no 'track' model. -->
+      <terrainHalfExtentX>60.0</terrainHalfExtentX>
+      <terrainHalfExtentY>60.0</terrainHalfExtentY>
       <wheelSpeedsTopicName>/ros_can/wheel_speeds</wheelSpeedsTopicName>
       <groundTruthWheelSpeedsTopicName>/ground_truth/wheel_speeds</groundTruthWheelSpeedsTopicName>

File: eufs_sim/eufs_racecar/robots/ads-dv/robot.urdf.xacro (robot description, xacro)
@@ -46,5 +46,5 @@
         <origin xyz="0.463 0.06792 0.224" rpy="0 0 0"/>
     </xacro:sensor_gps>
-    <xacro:VLP-16R parent="chassis" name="velodyne" topic="/velodyne_points" hz="10" samples="800" active="$(arg simulate_perception)">
+    <xacro:VLP-16R parent="chassis" name="velodyne" topic="/velodyne_points" hz="10" active="$(arg simulate_perception)">
 	    <origin xyz="0.243 0.0 0.324" rpy="0 ${6.1*M_PI/180.0} 0"/>
     </xacro:VLP-16R>

File: eufs_sim/eufs_racecar/robots/eufs/robot.urdf.xacro (robot description, xacro)
@@ -46,7 +46,8 @@
         <origin xyz="0.0 0.0 0.4" rpy="0 0 0"/>
     </xacro:sensor_gps>
-    <!-- Real car: VLP-16 (16 channels) mounted on the nose cone.
-         lasers must be passed explicitly — the VLP-16R macro default is 40. -->
-    <xacro:VLP-16R parent="chassis" name="velodyne" topic="/velodyne_points" hz="10" lasers="16" active="$(arg simulate_perception)">
+    <!-- Real car: VLP-16 (16 channels) mounted on the nose cone. hz is the only
+         knob; the macro derives horizontal resolution from it the way the
+         hardware does (10 Hz -> 0.2 deg). -->
+    <xacro:VLP-16R parent="chassis" name="velodyne" topic="/velodyne_points" hz="10" active="$(arg simulate_perception)">
         <origin xyz="1.6 0.0 0.25" rpy="0 ${1*M_PI/180.0} 0"/>
         <!-- main-hoop mount (previous): <origin xyz="-0.15 0.0 0.79" rpy="0 ${1*M_PI/180.0} 0"/> -->

File: eufs_sim/eufs_sensors/urdf/VLP-16R.urdf.xacro (robot description, xacro)
@@ -3,7 +3,17 @@
   <xacro:property name="M_PI" value="3.1415926535897931" />
   <!-- Real VLP-16 spec, not a cheaper approximation of one.
-       360 deg horizontal at 0.2 deg (the Puck's resolution at its 10 Hz
-       rotation) is 1800 samples per laser, 16 lasers, 28800 rays per rev,
-       288k points/s against the datasheet's ~300k.
+       Horizontal resolution is NOT a free parameter: the Puck fires each laser
+       on a fixed interval, so spinning faster spreads the same firings over
+       more degrees. The datasheet's table falls straight out of that, and the
+       giveaway is that points/second is constant across all three rates:
+         5 Hz -> 0.1 deg -> 3600 samples/rev -> 57600 pts/rev -> 288k pts/s
+        10 Hz -> 0.2 deg -> 1800 samples/rev -> 28800 pts/rev -> 288k pts/s
+        20 Hz -> 0.4 deg ->  900 samples/rev -> 14400 pts/rev -> 288k pts/s
+       So `hz` is the only knob, and samples follow: 360/(0.02*hz) = 18000/hz.
+       Carrying both independently lets them disagree, which is how ads-dv ended
+       up asking for 0.45 deg at 10 Hz, a sensor that does not exist.
+       Vertical is fixed by hardware and does not scale with rate: 16 lasers
+       over +/-15 deg at 2.0 deg. `lasers` defaulted to 40 here, 2.5x the real
+       count, and ads-dv silently took that default.
        This used to be 350 samples over 229 deg = 0.655 deg/ray, which is 3.3x
        coarser than the real sensor and 19 % of its rays. That made the sim
@@ -12,12 +22,13 @@
        It costs real time factor, and that is the right trade. Measured: RTF
        0.406, and every sensor still hits its configured rate IN SIM TIME, which
-       is the only clock perception, SLAM and planning read: cameras 30.30 and
-       29.85 Hz, velodyne 10.00, /cones 29.41. Wall clock is 2.5x slower and
-       nothing downstream can tell. Use scripts/measure_sim_rates.py, not
+       is the only clock perception, SLAM and planning read: both cameras 29.41
+       Hz, velodyne 10.00, /cones 10.00. Wall clock is 2.5x slower and nothing
+       downstream can tell. Use scripts/measure_sim_rates.py, not
        `ros2 topic hz`, which reports wall clock and will make this look broken.
-       Giving the LiDAR MORE rays also fixed the camera pair: at 0.655 deg/ray
-       the right camera sat at 20.00 Hz against the left's 29.41, and at spec
-       they run 30.30 / 29.85 together. More wall time per sim tick means both
-       renders finish. -->
+       An earlier version of this comment credited the ray count with fixing a
+       stereo rate split. There was no split. The "right camera at half rate"
+       came from probes that subscribed to both image streams from one Python
+       process, which cannot deserialise 2x 2.7 MB at 30 Hz; each camera reads
+       29.41 Hz when measured one topic per process. Measure that way. -->
   <xacro:macro
     name="VLP-16R"
@@ -26,6 +37,6 @@
             topic:=/velodyne_points
             hz:=10
-            lasers:=40
-            samples:=1800
+            lasers:=16
+            samples:=0
             min_range:=0.2
             max_range:=100.0
@@ -33,4 +44,9 @@
             min_angle:=-3.14159265
             max_angle:=3.14159265">
+    <!-- samples=0 means "be a real Puck at this rate". A non-zero value is an
+         explicit, knowing departure from the datasheet, not a default. -->
+    <xacro:property name="h_samples"
+                    value="${int(round(18000.0 / hz)) if samples == 0 else samples}"/>
+    <xacro:property name="h_res_deg" value="${360.0 / h_samples}"/>
     <joint name="${name}_base_mount_joint" type="fixed">
       <xacro:insert_block name="origin" />
@@ -92,6 +108,7 @@
           <ray>
             <scan>
+              <!-- ${h_samples} samples/rev = ${h_res_deg} deg at ${hz} Hz -->
               <horizontal>
-                <samples>${samples}</samples>
+                <samples>${h_samples}</samples>
                 <resolution>1.0</resolution>
                 <min_angle>${min_angle}</min_angle>

File: eufs_sim/eufs_sensors/urdf/zed.urdf.xacro (robot description, xacro)
@@ -102,11 +102,22 @@
     <xacro:unless value="${active}">
       <gazebo reference="${prefix}_left_camera_frame">
-        <sensor type="camera" name="${prefix}_left_camera">
-          <!-- see MultiSenseSLPlugin.h for available modes -->
+        <!-- ONE multicamera sensor, not two camera sensors. This is what makes
+             the pair a stereo pair.
+             As two independent sensors they each chased their own sim time
+             tick, and under load the right one missed every other tick and sat
+             at EXACTLY half the left's rate (15.15 against 28.99). Two images
+             at different sim instants are not a stereo pair: the disparity
+             between them contains the car's motion, not the scene's depth, and
+             the ZNCC cross check that removes the monocular tier's range bias
+             silently stops running.
+             A multicamera sensor renders both children in ONE update, so they
+             share a sim time and a stamp by construction rather than by luck.
+             Tuning rates could never have fixed this; it is structural. -->
+        <sensor type="multicamera" name="${prefix}_stereo_camera">
           <always_on>true</always_on>
           <update_rate>30.0</update_rate>
           <visualize>false</visualize>
-          <camera>
-            <pose>0 0.0 0 0 0 0</pose>
+          <camera name="left">
+            <pose>0 0.06 0 0 0 0</pose>
             <horizontal_fov>1.91986</horizontal_fov>
             <image>
@@ -125,35 +136,6 @@
             </noise>
           </camera>
-          <plugin name="${prefix}_left_camera_controller" filename="libgazebo_ros_camera.so">
-            <ros>
-              <parameter name="update_rate" type="double">30.0</parameter>
-              <remapping>/${prefix}_left/image_raw:=/${prefix}/left/image_rect_color</remapping>
-              <remapping>/${prefix}_left/camera_info:=/${prefix}/left/camera_info</remapping>
-              <qos>
-                <topic name="/${prefix}/left/image_rect_color">
-                  <publisher>
-                    <reliability>reliable</reliability>
-                  </publisher>
-                </topic>
-                <topic name="/${prefix}/left/camera_info">
-                  <publisher>
-                    <reliability>reliable</reliability>
-                  </publisher>
-                </topic>
-              </qos>
-            </ros>
-            <camera_name>${prefix}_left</camera_name>
-            <frame_name>${prefix}_left_camera_optical_frame</frame_name>
-            <triggered>false</triggered>
-          </plugin>
-        </sensor>
-      </gazebo>
-      <gazebo reference="${prefix}_right_camera_frame">
-        <sensor type="camera" name="${prefix}_right_camera">
-          <always_on>true</always_on>
-          <update_rate>30.0</update_rate>
-          <visualize>false</visualize>
-          <camera>
-            <pose>0 0.0 0 0 0 0</pose>
+          <camera name="right">
+            <pose>0 -0.06 0 0 0 0</pose>
             <horizontal_fov>1.91986</horizontal_fov>
             <image>
@@ -172,25 +154,12 @@
             </noise>
           </camera>
-          <plugin name="${prefix}_right_camera_controller" filename="libgazebo_ros_camera.so">
+          <plugin name="${prefix}_stereo_controller" filename="libgazebo_ros_camera.so">
             <ros>
-              <parameter name="update_rate" type="double">30.0</parameter>
-              <remapping>/${prefix}_right/image_raw:=/${prefix}/right/image_rect_color</remapping>
-              <remapping>/${prefix}_right/camera_info:=/${prefix}/right/camera_info</remapping>
-              <qos>
-                <topic name="/${prefix}/right/image_rect_color">
-                  <publisher>
-                    <reliability>reliable</reliability>
-                  </publisher>
-                </topic>
-                <topic name="/${prefix}/right/camera_info">
-                  <publisher>
-                    <reliability>reliable</reliability>
-                  </publisher>
-                </topic>
-              </qos>
+              <remapping>${prefix}/left/image_raw:=${prefix}/left/image_rect_color</remapping>
+              <remapping>${prefix}/right/image_raw:=${prefix}/right/image_rect_color</remapping>
             </ros>
-            <camera_name>${prefix}_right</camera_name>
-            <frame_name>${prefix}_right_camera_optical_frame</frame_name>
-            <triggered>false</triggered>
+            <camera_name>${prefix}</camera_name>
+            <frame_name>${prefix}_left_camera_optical_frame</frame_name>
+            <hack_baseline>0.12</hack_baseline>
           </plugin>
         </sensor>
