Commit message: perception: report the vision tiers' error ellipse, and measure what it costs
The tiers handed SLAM a circle. A vision cone's error is not one: at 15 m the
bearing is good to ~5 cm while the depth is good to ~2 m, and the ellipse's
major axis lies along the ray, not along x or y. One isotropic number was
simultaneously ~160x too pessimistic across the corridor and ~7x too optimistic
along it. SLAM already carries a full 2x2 landmark covariance and consumes what
perception reports, so the fix was to stop lying to it, not to build a tracker.

Both tiers work in the fraction sigma_D/D rather than absolute sigma_D, which is
what lets the model survive the optical-depth -> ground-range projection the
tiers have already applied by the time _cluster_to_cone sees the cluster.

LiDAR keeps its constants: it ranges directly to ~1%, so its error really is the
near-circle they describe.

Then build the instrument the roadmap asked for, and let it overrule the plan:

- Measure against /ground_truth/track, not /ground_truth/cones. The latter is
  FOV-filtered by the sim plugin, so recall against it plots the instrument's
  limit rather than the pipeline's. The gate is now ours: explicit, printed, and
  tunable. Truth outside it is excluded rather than counted as a false positive,
  so widening it cannot manufacture FPs.
- Cone identity for time-to-confirm is the plugin's link index, not a position
  hash. Cones are physics objects: the car knocks them and they move, and the
  plugin reports their live WorldPose, so a position key would mint a new
  identity for every nudged cone.
- Add covariance consistency (lat z^2 / lon z^2 / NEES). It was not in the plan
  and it turned out to be the acceptance test the whole thing needed.
- Add an end-to-end latency probe at /cones publish. Nothing measured latency
  before, which was untenable for a stack that lists it as a priority.

What the instrument then said, on small_track:

- sigma_d_px 0.25 was shipped as an admitted guess and measured lon z^2 = 0.96
  first time out. It was right.
- sigma_u_px 1.5 -> 3.0, from the stereo tier, whose errors sit far inside the
  match radius and so are not truncated by it.
- monocular NEES/2 went 138.58 -> 1.43; stereo 2.30 -> 1.11. Both vision tiers
  are now within ~2x of honest, and conservative in depth.

And it reversed Step 3. The plan was to delete the 16 px monocular cut, on the
argument that a far cone's bearing stays good and only its depth goes bad. That
is true of an ideal detector and false of this one. Lateral error by range:

    <= 8.8 m     implied sigma_u   1.0 - 2.6 px    the model holds exactly
    8.8 - 10 m   implied sigma_u   13.6 px
    10 - 20 m    implied sigma_u   17 - 32 px

The bearing collapses at ~9 m, inside one 1.25 m band, and the cliff survives
both a 1.0 m and a 2.0 m match radius. 9 m is where the cone is ~18 px at 720p:
~9 px at the detector's imgsz 640 input, about one stride-8 cell. Recall falls
off the same cliff (85% at 7.5-10 m, 14% at 12.5-15 m). Restoring the cut
dropped monocular lat z^2 from 260 to 10.7 with no other change.

So the cut sits on a real cliff in the detector, and it is the "trustworthy
range" boundary the pipeline is designed around: LiDAR clusters are the
backbone, and a camera-only cone is published only where its estimate can be
trusted. Step 4 (detector input resolution) is the prerequisite for Step 3, not
the other way round.

Also disable the ZED's depth sensor: a second full 1280x720 render pass plus a
point cloud, with /zed/depth/image_raw, /zed/points and /zed/image_raw all
measured at zero subscribers. Its effect on the camera rate is unmeasured and
the commit does not claim one.

Two things left honest rather than hidden: sigma_h_px 4.0 inflates noise to
cover a measured -0.88 m curve bias, which is a patch until c/e are re-fit; and
/cones runs at 4 Hz against a 10 Hz backbone with ~0.8 s latency because Tier 3
SIFT burns 200-235% CPU. That is the latency bomb 2.2 predicted, now gone off,
and it makes Step 5 a throughput fix rather than an accuracy one.

Co-Authored-By: Claude Opus 4.8 (1M context) <noreply@anthropic.com>

File: eufs_sim/eufs_sensors/urdf/zed.urdf.xacro (robot description, xacro)
@@ -3,5 +3,9 @@
   xmlns:xacro="http://www.ros.org/wiki/xacro">
   <xacro:property name="M_PI" value="3.1415926535897931" />
-  <xacro:macro name="zed_camera" params="prefix parent *origin active">
+  <!-- depth: emit the Gazebo `depth` sensor. Off by default because it costs a
+       second full 1280x720 render pass plus a point cloud, competing with the
+       left and right cameras for the render thread, and nothing in this
+       workspace subscribes to what it produces. See the block itself. -->
+  <xacro:macro name="zed_camera" params="prefix parent *origin active depth:=false">
     <joint name="${prefix}_base_joint" type="fixed">
       <axis xyz="1 0 0"/>
@@ -65,6 +69,14 @@
          or it drops the stereo tier for that frame, which starved Tier 3. Equal,
          sustainable rates keep both sensors on the same update tick.
-         The depth camera is not subscribed by anything in this workspace, so it only
-         competed for the GPU; it is kept alive at a token rate. -->
+         MEASURED AGAIN, and the ceiling is lower than it looks: at a 30 Hz request
+         the left camera achieved 8.9 Hz while the right achieved 17.2 Hz: they
+         diverged, which is the same starvation, so 30 is not available here. At 15
+         both settle at ~8.8 Hz together, which is why 15 stays. The GPU is not the
+         limit (gzserver renders on the RTX 4070 at ~150% CPU); Gazebo Classic
+         serialises every sensor on one render thread, so the two cameras and the
+         12800-ray VLP-16 share it. To go faster, cut that work, not the request.
+         The depth camera is not subscribed by anything in this workspace, so it
+         only competed for the render thread; it is now off by default (depth false)
+         rather than kept alive at a token rate. -->
     <!-- Simulate raw perception sensors only if we're not using the abstracted perception simulation -->
     <xacro:unless value="${active}">
@@ -74,5 +86,5 @@
           <always_on>true</always_on>
           <update_rate>15.0</update_rate>
-          <visualize>true</visualize>
+          <visualize>false</visualize>
           <camera>
             <pose>0 0.0 0 0 0 0</pose>
@@ -121,5 +133,5 @@
           <always_on>true</always_on>
           <update_rate>15.0</update_rate>
-          <visualize>true</visualize>
+          <visualize>false</visualize>
           <camera>
             <pose>0 0.0 0 0 0 0</pose>
@@ -164,6 +176,18 @@
         </sensor>
       </gazebo>
+      <!-- Depth simulation. DISABLED.
+           A `depth` sensor costs a full 1280x720 render pass plus a point
+           cloud, and nothing subscribes to any of what it emits:
+           /zed/depth/image_raw, /zed/points and /zed/image_raw all measured
+           zero subscribers with the real perception stack running. The stereo
+           tier works from the left and right image_rect_color topics instead.
+           The cost is not the 1 Hz it asks for: it competes with the left and
+           right cameras for Gazebo's render thread, and those two already miss
+           their requested rate (15 Hz asked, ~8.8 Hz achieved), which is what
+           starves the bbox/LiDAR pairing downstream.
+           Re-enable (always_on true) only if something actually consumes it,
+           e.g. if the ZED SDK NEURAL depth option in the roadmap is tried. -->
+      <xacro:if value="${depth}">
       <gazebo reference="${prefix}_depth_camera_frame">
-        <!-- Depth simulation -->
         <sensor name="stereo_depth" type="depth">
           <always_on>true</always_on>
@@ -196,4 +220,5 @@
         </sensor>
       </gazebo>
+      </xacro:if>
     </xacro:unless>
   </xacro:macro>
