Commit message: sim: teach every sensor its real error structure, and ship the harness to pin it
The 4WD AMK chain (18-bit encoder -> int16 motor rpm / gear ratio), slip
from achieved dynamics, colored INS errors with believed-not-realized
covariance, transport latency, the lidar realism bridge (motion
distortion, ground dropout, real driver layout), dead sensor cleanup,
and sensor_parity_report.py so every estimate here can be pinned against
real logs. The -2 cm gpu_ray 'ground bias' and the 20 Hz right camera
both closed as measurement-era artifacts, with the receipts in-tree.

Co-Authored-By: Claude Fable 5 <noreply@anthropic.com>

File: eufs_sim/eufs_racecar/robots/ads-dv/robot.urdf.xacro (robot description, xacro)
@@ -37,5 +37,4 @@
     <!--     LOCATIONS: (XYZ)
     IMU: 0.0 0.0 0.0
-    GPS: 0.463 0.0679 0.224
     LIDAR: 0.243 0.0 0.324
     STEREO CAM: 0.334 0.0 0.295 -->
@@ -43,8 +42,8 @@
         <origin xyz="0.0 0.0 0.0" rpy="0 0 0"/>
     </xacro:sensor_imu>
-    <xacro:sensor_gps parent="chassis" prefix="gps">
-        <origin xyz="0.463 0.06792 0.224" rpy="0 0 0"/>
-    </xacro:sensor_gps>
-    <xacro:VLP-16R parent="chassis" name="velodyne" topic="/velodyne_points" hz="10" active="$(arg simulate_perception)">
+    <!-- No gazebo GPS/magnetometer/zed_imu: zero subscribers; the GNSS/INS
+         path is sim_ellipse_d at the driver level. See robots/eufs. -->
+    <!-- Ideal scan; the lidar_realism bridge owns /velodyne_points. -->
+    <xacro:VLP-16R parent="chassis" name="velodyne" topic="/velodyne_points_ideal" hz="10" active="$(arg simulate_perception)">
 	    <origin xyz="0.243 0.0 0.324" rpy="0 ${6.1*M_PI/180.0} 0"/>
     </xacro:VLP-16R>
@@ -52,9 +51,3 @@
 	    <origin xyz="0.334 0.0 0.295" rpy="0 ${10.15*M_PI/180.0} 0"/>
     </xacro:zed_camera>
-    <xacro:sensor_imu parent="chassis" prefix="zed_imu" topic_prefix="/camera">
-        <origin xyz="0.334 0.0 0.295" rpy="0 ${10.15*M_PI/180.0} 0"/>
-    </xacro:sensor_imu>
-    <xacro:sensor_magnetometer parent="chassis" prefix="sbg">
-        <origin xyz="0.0 0.0 0.0" rpy="0 0 0"/>
-    </xacro:sensor_magnetometer>
 </robot>

File: eufs_sim/eufs_racecar/robots/eufs/robot.urdf.xacro (robot description, xacro)
@@ -37,5 +37,4 @@
     <!--     LOCATIONS: (XYZ)
     IMU: 0.0 0.0 0.170
-    GPS: -0.110 0.0 0.9
     LIDAR: 1.700 0.0 -0.150
     STEREO CAM: -0.110 0.0 0.800 -->
@@ -43,11 +42,18 @@
         <origin xyz="0.0 0.0 0.0" rpy="0 0 0"/>
     </xacro:sensor_imu>
-    <xacro:sensor_gps parent="chassis" prefix="gps">
-        <origin xyz="0.0 0.0 0.4" rpy="0 0 0"/>
-    </xacro:sensor_gps>
+    <!-- No gazebo GPS or magnetometer. Nothing in the stack consumed either
+         topic, and the GNSS/INS path is simulated at the driver level by
+         sim_ellipse_d (/sbg/ekf_nav + /sbg/ekf_euler), where the Ellipse-D
+         error model actually lives. A raw 2 m-white-noise NavSatFix next to
+         a cm-level RTK model was only there to mislead. -->
     <!-- Real car: VLP-16 (16 channels) mounted on the nose cone. hz is the only
          knob; the macro derives horizontal resolution from it the way the
-         hardware does (10 Hz -> 0.2 deg). -->
-    <xacro:VLP-16R parent="chassis" name="velodyne" topic="/velodyne_points" hz="10" active="$(arg simulate_perception)">
+         hardware does (10 Hz -> 0.2 deg).
+         The sensor emits the geometrically ideal scan on _ideal; the
+         lidar_realism bridge (spawned by load_car.launch.py) owns
+         /velodyne_points, adding motion distortion, far-ground dropout and
+         the real driver's ring/time field layout. Its spin_hz must match
+         hz here. -->
+    <xacro:VLP-16R parent="chassis" name="velodyne" topic="/velodyne_points_ideal" hz="10" active="$(arg simulate_perception)">
         <origin xyz="1.6 0.0 0.25" rpy="0 ${1*M_PI/180.0} 0"/>
         <!-- main-hoop mount (previous): <origin xyz="-0.15 0.0 0.79" rpy="0 ${1*M_PI/180.0} 0"/> -->
@@ -56,9 +62,5 @@
         <origin xyz="-0.08 0.0 0.76" rpy="0 0 0"/>
     </xacro:zed_camera>
-    <xacro:sensor_imu parent="chassis" prefix="zed_imu" topic_prefix="/camera">
-        <origin xyz="-0.08 0.0 0.76" rpy="0 0 0"/>
-    </xacro:sensor_imu>
-    <xacro:sensor_magnetometer parent="chassis" prefix="sbg">
-        <origin xyz="0.0 0.0 0.0" rpy="0 0 0"/>
-    </xacro:sensor_magnetometer>
+    <!-- No zed_imu: the ZED's built-in IMU is not used by the stack, and its
+         simulated stream (/camera/imu/data) had zero subscribers. -->
 </robot>

File: eufs_sim/eufs_sensors/urdf/VLP-16R.urdf.xacro (robot description, xacro)
@@ -46,9 +46,11 @@
        behind them. That, not texel resolution, was the bulk of the "gpu_ray
        quality is terrible" symptom; the staircase was the rest. Known
-       residuals vs CPU ray, measured and accepted: ground reads ~2 cm low
-       (constant height offset, root cause not yet found; cones unaffected at
-       +4 mm radial), car-body self-returns differ (visual vs collision
-       geometry — crop them like on the real car), and the -3 deg ring keeps
-       a ~2x-noise staircase (grazing-incidence limit of the method). -->
+       residuals vs CPU ray, measured and accepted: car-body self-returns
+       differ (visual vs collision geometry — crop them like on the real
+       car), and the -3 deg ring keeps a ~2x-noise staircase
+       (grazing-incidence limit of the method). The old "ground reads ~2 cm
+       low" residual was resolved 2026-07-16: it was the CAR settling at a
+       different height per run, not the sensor — see the Known residuals
+       section of tools/gazebo-patches/README.md for the measurements. -->
   <xacro:macro
     name="VLP-16R"

File: eufs_sim/eufs_sensors/urdf/all_sensors.urdf.xacro (robot description, xacro)
@@ -1,11 +1,12 @@
 <?xml version="1.0"?>
 <robot name="all_sensors" xmlns:xacro="http://www.ros.org/wiki/xacro">
-  <!-- This file unifies all sensors that can be used on simulation, defined as xacro:macros -->
-  <!-- GPS -->
-  <xacro:include filename="$(find eufs_sensors)/urdf/gps.urdf.xacro"/>
+  <!-- This file unifies all sensors that can be used on simulation, defined
+       as xacro:macros.
+       Gone, deliberately: the gazebo GPS and magnetometer macros. Nothing
+       subscribed to either topic, and the GNSS/INS chain is simulated at the
+       driver level by scripts/sim_ellipse_d.py (/sbg/ekf_nav + ekf_euler),
+       which carries the Ellipse-D error model the raw sensors never had. -->
   <!-- Velodyne VLP-16R -->
   <xacro:include filename="$(find eufs_sensors)/urdf/VLP-16R.urdf.xacro"/>
-  <!-- Magnetometer-->
-  <xacro:include filename="$(find eufs_sensors)/urdf/magnetometer.urdf.xacro"/>
   <!--IMU -->
   <xacro:include filename="$(find eufs_sensors)/urdf/imu.urdf.xacro"/>

File: eufs_sim/eufs_sensors/urdf/imu.urdf.xacro (robot description, xacro)
@@ -1,5 +1,53 @@
 <?xml version="1.0"?>
 <robot name="sensor_imu" xmlns:xacro="http://www.ros.org/wiki/xacro">
-    <xacro:macro name="sensor_imu" params="prefix parent topic_prefix *origin noise:=0.08">
+    <!-- Simulated SBG Ellipse-D IMU stream (what the sbg driver puts on
+         `imu/data`), replacing the stock EUFS model.
+         This used to be a single `noise:=0.08` applied to BOTH the gyro
+         [rad/s] and the accelerometer [m/s^2]: one number for two different
+         physical units, and the wrong magnitude for either. 0.08 rad/s is
+         4.6 deg/s of white noise per sample - roughly 60x the real Ellipse-D
+         gyro at a 200 Hz output - and it carried no bias at all. Both errors
+         matter downstream in opposite directions: wheel_odometry.py consumes
+         this topic's yaw rate, so its sim behaviour was driven by a heading
+         random walk of ~0.15 deg/sqrt(s) (the real unit: 0.003), while the
+         missing bias made long dead-reckoning look better than a real gyro
+         ever is (white noise averages out; bias integrates linearly).
+         The knobs are physical densities, not per-sample sigmas; the
+         per-sample stddev follows the output rate the way the hardware does:
+         sigma = density * sqrt(rate). Change `hz` and the noise power stays
+         physical; correct a datasheet number and it is a one-value edit.
+         Datasheet values (Ellipse-D, MK068EN - the same source
+         sim_ellipse_d.py quotes for its INS error model):
+           gyro angular random walk  0.18 deg/sqrt(h) = 5.24e-5 rad/s/sqrt(Hz)
+           gyro in-run bias          7 deg/h          = 3.4e-5  rad/s
+           accel noise density       57 ug/sqrt(Hz)   = 5.6e-4  m/s^2/sqrt(Hz)
+           accel in-run bias         14 ug            = 1.4e-4  m/s^2
+           imu/data output rate      200 Hz (was 1000 here - 5x the driver)
+         What gazebo classic does with these: white noise per sample, plus ONE
+         bias per axis drawn at startup from N(bias_mean, bias_stddev) with a
+         random sign, held for the whole run. That is a turn-on/in-run bias
+         *level*, not a bias walk - classic ignores SDF's dynamic_bias_* tags.
+         Over a single 2-10 min session a fixed draw at the in-run instability
+         level is the honest first-order model; if slow bias wander ever
+         matters, it needs a post-processing node (sim_ellipse_d.py already
+         carries these constants for its own dead-reckoning model).
+         TRAP, recorded for future consumers: the `orientation` field of the
+         published Imu message carries NO noise. Gazebo classic only perturbs
+         rates and accelerations, so orientation is ground truth - a free
+         perfect AHRS that does not exist on the car. Nothing may consume sim
+         /imu/data orientation as if it were a real attitude estimate; use
+         /sbg/ekf_euler from sim_ellipse_d, which degrades honestly.
+         wheel_odometry.py reads only angular_velocity.z and is safe. -->
+    <xacro:macro name="sensor_imu"
+                 params="prefix parent topic_prefix *origin
+                         hz:=200
+                         gyro_noise_density:=5.24e-5
+                         gyro_bias_stddev:=3.4e-5
+                         accel_noise_density:=5.6e-4
+                         accel_bias_stddev:=1.4e-4">
+        <xacro:property name="gyro_stddev"
+                        value="${float(gyro_noise_density) * (float(hz) ** 0.5)}"/>
+        <xacro:property name="accel_stddev"
+                        value="${float(accel_noise_density) * (float(hz) ** 0.5)}"/>
         <joint name="${prefix}_base_joint" type="fixed">
             <axis xyz="1 0 0"/>
@@ -8,14 +56,20 @@
             <child link="${prefix}_base_link"/>
         </joint>
+        <!-- Ellipse-D-class body: 65 g, 46x45x32 mm, inertia consistent with
+             that box (the old 1 mm/1 g link carried 0.1 g-m^2 inertias, 1e6x
+             its own physics). Lumped into the chassis by the fixed joint
+             either way; this is about not asserting absurd numbers. -->
         <link name="${prefix}_base_link">
             <inertial>
-                <mass value="0.001"/>
+                <mass value="0.065"/>
                 <origin rpy="0 0 0" xyz="0 0 0"/>
-                <inertia ixx="0.0001" ixy="0" ixz="0" iyy="0.000001" iyz="0" izz="0.0001"/>
+                <inertia ixx="${0.065/12.0*(0.045*0.045+0.032*0.032)}" ixy="0" ixz="0"
+                         iyy="${0.065/12.0*(0.046*0.046+0.032*0.032)}" iyz="0"
+                         izz="${0.065/12.0*(0.046*0.046+0.045*0.045)}"/>
             </inertial>
             <visual>
                 <origin rpy="0 0 0" xyz="0 0 0"/>
                 <geometry>
-                    <box size="0.001 0.001 0.001"/>
+                    <box size="0.046 0.045 0.032"/>
                 </geometry>
             </visual>
@@ -23,5 +77,5 @@
                 <origin rpy="0 0 0" xyz="0 0 0"/>
                 <geometry>
-                    <box size=".001 .001 .001"/>
+                    <box size="0.046 0.045 0.032"/>
                 </geometry>
             </collision>
@@ -29,9 +83,8 @@
         <gazebo reference="${prefix}_base_link">
             <gravity>true</gravity>
-            <sensor name="{prefix}_sensor" type="imu">
+            <sensor name="${prefix}_sensor" type="imu">
                 <always_on>true</always_on>
-                <update_rate>1000</update_rate>
-                <visualize>true</visualize>
-                <topic>imu/data</topic>
+                <update_rate>${hz}</update_rate>
+                <visualize>false</visualize>
                 <imu>
                     <angular_velocity>
@@ -39,5 +92,7 @@
                             <noise type="gaussian">
                                 <mean>0.0</mean>
-                                <stddev>${noise}</stddev>
+                                <stddev>${gyro_stddev}</stddev>
+                                <bias_mean>0.0</bias_mean>
+                                <bias_stddev>${gyro_bias_stddev}</bias_stddev>
                             </noise>
                         </x>
@@ -45,5 +100,7 @@
                             <noise type="gaussian">
                                 <mean>0.0</mean>
-                                <stddev>${noise}</stddev>
+                                <stddev>${gyro_stddev}</stddev>
+                                <bias_mean>0.0</bias_mean>
+                                <bias_stddev>${gyro_bias_stddev}</bias_stddev>
                             </noise>
                         </y>
@@ -51,5 +108,7 @@
                             <noise type="gaussian">
                                 <mean>0.0</mean>
-                                <stddev>${noise}</stddev>
+                                <stddev>${gyro_stddev}</stddev>
+                                <bias_mean>0.0</bias_mean>
+                                <bias_stddev>${gyro_bias_stddev}</bias_stddev>
                             </noise>
                         </z>
@@ -59,5 +118,7 @@
                             <noise type="gaussian">
                                 <mean>0.0</mean>
-                                <stddev>${noise}</stddev>
+                                <stddev>${accel_stddev}</stddev>
+                                <bias_mean>0.0</bias_mean>
+                                <bias_stddev>${accel_bias_stddev}</bias_stddev>
                             </noise>
                         </x>
@@ -65,5 +126,7 @@
                             <noise type="gaussian">
                                 <mean>0.0</mean>
-                                <stddev>${noise}</stddev>
+                                <stddev>${accel_stddev}</stddev>
+                                <bias_mean>0.0</bias_mean>
+                                <bias_stddev>${accel_bias_stddev}</bias_stddev>
                             </noise>
                         </y>
@@ -71,5 +134,7 @@
                             <noise type="gaussian">
                                 <mean>0.0</mean>
-                                <stddev>${noise}</stddev>
+                                <stddev>${accel_stddev}</stddev>
+                                <bias_mean>0.0</bias_mean>
+                                <bias_stddev>${accel_bias_stddev}</bias_stddev>
                             </noise>
                         </z>

File: eufs_sim/eufs_sensors/urdf/zed.urdf.xacro (robot description, xacro)
@@ -94,9 +94,20 @@
          camera noise (faster, but the detector trains on FSOCO's real noisy
          images, so a clean sim is an easier sim).
-         KNOWN AND OPEN: the right camera settles at 20.00 Hz in sim time while
-         the left holds 29.41, and both jitter badly (60 to 100 ms against the
-         velodyne's 0.3). The ZNCC cross check needs both images within
-         max_image_age_sec or it silently does not run, and it is what removes
-         the monocular tier's range bias. Watch its confirm rate. -->
+         RESOLVED 2026-07-16 (was KNOWN AND OPEN: right camera at 20.00 Hz,
+         both jittering 60-100 ms). Re-measured headless on the current stack
+         (patched gazebo, gpu_ray TEX 8192, R8G8B8, __GL_YIELD), one topic
+         per process, stamps in sim time:
+           sensors-only:       left 30.00 Hz, right 30.00 Hz
+           full stack (YOLO):  left 30.00 Hz, right 30.00 Hz, inter-stamp
+                               sigma 0.9 ms (a 33/34 ms alternation - the
+                               1 ms physics step quantizing 33.33 ms), and
+                               751/751 overlapping frames share their stamp
+                               bit-exactly between left and right.
+         The old symptom belonged to the era of the CPU-ray LiDAR starving
+         the render thread. The structural guarantee the ZNCC cross check
+         needs (one multicamera update = one shared stamp) measures true; it
+         still silently skips pairs older than max_image_age_sec, so if its
+         confirm rate ever drops again, re-run this measurement before
+         touching any rates. -->
     <!-- Simulate raw perception sensors only if we're not using the abstracted perception simulation -->
     <xacro:unless value="${active}">
