Commit message: sim: in-render camera realism + per-launch calibration residuals
Camera realism moved INTO the render path: gazebo_camera_realism
subclasses the stock gazebo_ros_camera and applies rolling-shutter skew
(readout 20 ms) plus exposure motion blur (4 ms, K remap taps) to the
frame buffer before publication, with the body twist read straight from
physics. The earlier topic-shim prototype halved the image rate and its
latency pushed YOLO bboxes past the perception pairing window; in-render
costs no extra hop and image_rect_color stays the only camera topic.
Flow model: rotational flow + FOE looming with a ground-plane depth
prior; gate symmetry/verification unaffected. Known limit: the ego
bodywork blurs like the world.

Calibration residuals, drawn FRESH each launch (real recalibration =
a new rig error): the physical sensors spawn at nominal + a random
ChArUco-class draw (camera/lidar mounts ~0.12 deg / 4-5 mm per axis,
stereo right-eye rectification ~0.03 deg) while TF keeps publishing the
nominal frames — exactly how a residual behaves on the car. Sigmas sized
to our rig (stereo self-rectification + lidar-camera board, 12 cm
squares). calib_seed reproduces a draw, calib_error:=false is the ideal
rig; every draw is logged by load_car.

ZED far clip 20 -> 300 m (the sky was clipped to a bare gradient;
SkyX clouds still need a gzclient-only shader fix, noted for the
gazebo-patches backlog).

Co-Authored-By: Claude Fable 5 <noreply@anthropic.com>

File: sim/eufs_sim/eufs_sensors/urdf/VLP-16R.urdf.xacro (robot description, xacro)
@@ -1,4 +1,6 @@
 <?xml version="1.0"?>
 <robot xmlns:xacro="http://www.ros.org/wiki/xacro" name="VLP-16">
+  <!-- Fresh per-launch draw from load_car.launch.py; default = ideal. -->
+  <xacro:arg name="calib_lidar_err" default="0 0 0 0 0 0"/>
   <xacro:property name="M_PI" value="3.1415926535897931" />
   <!-- Real VLP-16 spec, not a cheaper approximation of one.
@@ -126,5 +128,10 @@
         <sensor type="${'gpu_ray' if str(gpu).lower() in ('true', '1') else 'ray'}" name="${name}-VLP16">
           <always_on>true</always_on>
-          <pose>0 0 0 0 0 0</pose>
+          <!-- Mount calibration residual: the PHYSICAL lidar sits at nominal
+               + this offset while TF keeps the nominal frame — the error a
+               real ChArUco-board (12 cm squares) lidar-camera calibration
+               leaves behind. Drawn fresh per launch in load_car.launch.py;
+               see zed.urdf.xacro for the camera-side residual. -->
+          <pose>$(arg calib_lidar_err)</pose>
           <visualize>false</visualize>
           <update_rate>${hz}</update_rate>

File: sim/eufs_sim/eufs_sensors/urdf/zed.urdf.xacro (robot description, xacro)
@@ -3,4 +3,15 @@
   xmlns:xacro="http://www.ros.org/wiki/xacro">
   <xacro:property name="M_PI" value="3.1415926535897931" />
+  <!-- Calibration residual (sim-to-real): the PHYSICAL sensors sit at
+       nominal + these offsets while every TF/projection keeps consuming the
+       nominal frames — exactly the error a real calibration leaves behind.
+       The values arrive from load_car.launch.py, which draws a FRESH
+       residual per launch (sigma calibrated to our rig: stereo
+       self-rectification + lidar-camera ChArUco board with 12 cm squares)
+       and logs the draw. Defaults are the ideal rig. -->
+  <xacro:arg name="calib_cam_err" default="0 0 0 0 0 0"/>
+  <xacro:arg name="calib_stereo_err_rpy" default="0 0 0"/>
+  <xacro:property name="zed_mount_err" value="$(arg calib_cam_err)"/>
+  <xacro:property name="zed_stereo_err_rpy" value="$(arg calib_stereo_err_rpy)"/>
   <!-- depth: emit the Gazebo `depth` sensor. Off by default because it costs a
        second full 1280x720 render pass plus a point cloud, competing with the
@@ -129,4 +140,6 @@
           <update_rate>30.0</update_rate>
           <visualize>false</visualize>
+          <!-- Rig mount calibration residual (see the property block). -->
+          <pose>${zed_mount_err}</pose>
           <!-- Poses are RELATIVE to the sensor's reference link, which is
                already the LEFT camera frame (y=+0.06 from center). The old
@@ -146,5 +159,10 @@
             <clip>
               <near>0.5</near>
-              <far>20</far>
+              <!-- 300, not 20: the SkyX cloud layer lives hundreds of
+                   meters up and a 20 m far plane culled it, so the camera
+                   only ever saw the bare gradient — an unrealistically
+                   clean YOLO background. Track geometry past 20 m is a few
+                   cones; the render cost is negligible. -->
+              <far>300</far>
             </clip>
             <noise>
@@ -155,5 +173,7 @@
           </camera>
           <camera name="right">
-            <pose>0 -0.12 0 0 0 0</pose>
+            <!-- Stereo rectification residual on the right eye (rotation
+                 only): biases ZNCC disparity like an imperfect self-calib. -->
+            <pose>0 -0.12 0 ${zed_stereo_err_rpy}</pose>
             <horizontal_fov>1.91986</horizontal_fov>
             <image>
@@ -164,5 +184,10 @@
             <clip>
               <near>0.5</near>
-              <far>20</far>
+              <!-- 300, not 20: the SkyX cloud layer lives hundreds of
+                   meters up and a 20 m far plane culled it, so the camera
+                   only ever saw the bare gradient — an unrealistically
+                   clean YOLO background. Track geometry past 20 m is a few
+                   cones; the render cost is negligible. -->
+              <far>300</far>
             </clip>
             <noise>
@@ -172,5 +197,9 @@
             </noise>
           </camera>
-          <plugin name="${prefix}_stereo_controller" filename="libgazebo_ros_camera.so">
+          <!-- Stock gazebo_ros_camera subclass: rolling-shutter skew and
+               exposure motion blur are applied to the render buffer INSIDE
+               the publish path (zero extra hop/latency; body twist read
+               straight from physics). See eufs_plugins/gazebo_camera_realism. -->
+          <plugin name="${prefix}_stereo_controller" filename="libgazebo_camera_realism.so">
             <ros>
               <remapping>${prefix}/left/image_raw:=${prefix}/left/image_rect_color</remapping>
@@ -180,4 +209,11 @@
             <frame_name>${prefix}_left_camera_optical_frame</frame_name>
             <hack_baseline>0.12</hack_baseline>
+            <motionBlur>true</motionBlur>
+            <rollingShutter>true</rollingShutter>
+            <exposureTime>0.004</exposureTime>
+            <readoutTime>0.020</readoutTime>
+            <blurTaps>3</blurTaps>
+            <cameraHeight>0.85</cameraHeight>
+            <horizontalFov>1.91986</horizontalFov>
           </plugin>
         </sensor>
